File: pcb/DinoSpand_v2.0/inputoutput.kicad_sch (KiCad schematic)
At the start: 34 parts, among them J4 Conn_01x02_Pin, J5 Conn_01x02_Pin, K1 EE2-5NU, K2 EE2-5NU, K3 EE2-5NU, K4 EE2-5NU, Q1 DMN62D0U-7, Q2 DMN62D0U-7, Q3 DMN62D0U-7, Q4 DMN62D0U-7

Commit message: pcbs update
Connections:
- net GND: now also Q1.2 (S), Q2.2 (S), Q3.2 (S), Q4.2 (S); no longer Q1.3 (S), Q2.3 (S), Q3.3 (S), Q4.3 (S)
- net at R2.2, R3.2: now also Q1.1 (G); no longer Q1.2 (G)
- net at D2.2 (A), K2.8: now also Q2.3 (D); no longer Q2.1 (D)
- net at D3.2 (A), K3.8: now also Q3.3 (D); no longer Q3.1 (D)
- net at R10.2, R11.2: now also Q3.1 (G); no longer Q3.2 (G)
- net at R14.2, R15.2: now also Q4.1 (G); no longer Q4.2 (G)
- net at R5.2, R6.2: now also Q2.1 (G); no longer Q2.2 (G)
- net at D1.2 (A), K1.8: now also Q1.3 (D); no longer Q1.1 (D)
- net at D6.2 (A), K4.8: now also Q4.3 (D); no longer Q4.1 (D)
