File: pcb/DinoSpand_v2.0/power.kicad_sch (KiCad schematic)
At the start: 9 parts, among them U3 LT1963AEST-3.3#TRPBF

Commit message: pcbs update
Parts:
- added C10: xuF, Capacitor_THT:CP_Radial_D4.0mm_P2.00mm, symbol Device:C
- added C11, C14, C15: xuF, Capacitor_SMD:C_0603_1608Metric, symbol Device:C
- added C12, C13: 10uF, Capacitor_SMD:C_0603_1608Metric, symbol Device:C
- added U4: LT1963AEST-3.3#TRPBF, Samacsys:SOT230P700X180-4N, symbol Samacsys:LT1963AEST-3.3#TRPBF
- C4, C9: footprint Capacitor_SMD:C_0603_1608Metric -> Capacitor_THT:CP_Radial_D4.0mm_P2.00mm
- D16: footprint LED_THT:LED_D3.0mm -> LED_SMD:LED_0603_1608Metric
Connections:
- net +3V3: now also C13.1, C14.1, C15.1, U4.3 (OUT)
- net GND: now also C10.2, C11.2, C12.2, C13.2, C14.2, C15.2, U4.2 (GND_1), U4.4 (GND_2)
- new net +5V: C10.1, C11.1, C12.1, U4.1 (IN)
Other:
- moved on the sheet: C4, C5, C6, C7, C8, C9, D16, R31, U3
