File: pcb/DinoSpand_v2.0/microcontroller.kicad_sch (KiCad schematic)
At the start: 12 parts, among them J6 Conn_01x04_Pin, U2 ESP32-S3-WROOM-1-N4

Commit message: pcbs update
Connections:
- net +3V3: no longer D12.1 (K)
- new net +5V: D12.1 (K)
Changed lines of the file:
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@@
 			)
 		)
-		(property "Value" "+3V3"
+		(property "Value" "+5V"
 			(at 104.14 119.38 0)
 			(effects

Commit message: pcbs final update
Parts:
- added D17: LED, LED_THT:LED_D3.0mm, symbol Device:LED
- added R32: 100, Resistor_SMD:R_0603_1608Metric, symbol Device:R
Connections:
- net GND: now also D17.1 (K)
- net GPIO39: now also R32.1
- new net: D17.2 (A), R32.2
- no-connect marks 11 -> 10
