File: pcb/DinoSpand_v2.0/DinoSpand_v2.0.kicad_pcb (KiCad board)
At the start: 2 copper layers, 70 x 59 mm, 80 parts, among them J1 Conn_01x04_Pin, J10 Conn_01x02_Pin, J11 3-794619-8, J2 Conn_01x02_Pin, J3 4-794619-6, J4 Conn_01x02_Pin, J5 Conn_01x02_Pin, J6 Conn_01x04_Pin, J7 Conn_01x02_Pin, J8 Conn_01x02_Pin, J9 Conn_01x02_Pin, K1 EE2-5NU, K2 EE2-5NU, K3 EE2-5NU, K4 EE2-5NU, Q1 DMN62D0U-7, Q2 DMN62D0U-7, Q3 DMN62D0U-7, Q4 DMN62D0U-7, U1 Oled64x128, U2 ESP32-S3-WROOM-1-N4, U3 LT1963AEST-3.3#TRPBF

Commit message: pcbs update
Parts:
- added C10: xuF, Capacitor_THT:CP_Radial_D4.0mm_P2.00mm, F.Cu at (152.0, 41.5)
- added C11: xuF, Capacitor_SMD:C_0603_1608Metric, F.Cu at (148.0, 47.0)
- added C12: 10uF, Capacitor_SMD:C_0603_1608Metric, F.Cu at (148.0, 44.5)
- added C13: 10uF, Capacitor_SMD:C_0603_1608Metric, B.Cu at (141.9, 44.2)
- added C14: xuF, Capacitor_SMD:C_0603_1608Metric, B.Cu at (142.0, 47.0)
- added C15: xuF, Capacitor_SMD:C_0603_1608Metric, B.Cu at (142.0, 49.5)
- added U4: LT1963AEST-3.3#TRPBF, Samacsys:SOT230P700X180-4N, B.Cu at (147.5, 46.9)
- C4, C9: footprint Capacitor_SMD:C_0603_1608Metric -> Capacitor_THT:CP_Radial_D4.0mm_P2.00mm
- D16: footprint LED_THT:LED_D3.0mm -> LED_SMD:LED_0603_1608Metric
- moved C9 5.47 mm to (152.7, 69.5), turned to -90 degrees
- moved D12 5.08 mm to (130.0, 41.5), turned to 180 degrees
- moved D16 4.30 mm to (156.0, 68.2), turned to 180 degrees
- moved C4 3.05 mm to (158.5, 85.8)
- moved C5 2.00 mm to (158.1, 82.5)
- moved R31 1.39 mm to (156.0, 68.2)
- moved J2 0.50 mm to (148.5, 67.7)
- moved C8 0.26 mm to (158.0, 70.5), turned to 0 degrees
- moved J1 0.25 mm to (148.5, 54.2)
- moved C7 0.07 mm to (158.0, 72.0), turned to 0 degrees
Connections:
- D12 pad 1: +3V3 -> +5V
- Q1 pad 1: Net-(D1-A) -> Net-(Q1-G)
- Q1 pad 2: Net-(Q1-G) -> GND
- Q1 pad 3: GND -> Net-(D1-A)
- Q2 pad 1: Net-(D2-A) -> Net-(Q2-G)
- Q2 pad 2: Net-(Q2-G) -> GND
- Q2 pad 3: GND -> Net-(D2-A)
- Q3 pad 1: Net-(D3-A) -> Net-(Q3-G)
- Q3 pad 2: Net-(Q3-G) -> GND
- Q3 pad 3: GND -> Net-(D3-A)
- Q4 pad 1: Net-(D6-A) -> Net-(Q4-G)
- Q4 pad 2: Net-(Q4-G) -> GND
- Q4 pad 3: GND -> Net-(D6-A)
Routing:
- net +5V: track 0.00 -> 31.9 mm, vias 0 -> 1
- net +3V3: track 146.3 -> 152.4 mm
- net GND: track 0.00 -> 5.40 mm, vias 421 -> 366
- net Net-(D1-A): track 20.6 -> 24.5 mm
- net Net-(D16-A): track 3.64 -> 0.02 mm, vias 0 -> 1
- net Net-(D2-A): track 26.0 -> 28.2 mm
- net /Microcontroller/GPIO5: track 28.1 -> 29.8 mm
- net Net-(D3-A): track 33.6 -> 34.8 mm
- net Net-(D12-A): track 4.56 -> 5.72 mm
- net /Microcontroller/GPIO6: track 35.0 -> 34.1 mm
- net /Microcontroller/GPIO16: track 42.5 -> 42.0 mm, vias 2 -> 1
- net /Microcontroller/GPIO15: vias 3 -> 2
- added copper zone on B.Cu, net +3V3
- added copper zone on F.Cu, net +3V3
- added copper zone on F.Cu, net Net-(D1-A)
- added copper zone on F.Cu, net Net-(D2-A)
- added copper zone on F.Cu, net Net-(D3-A)
- added copper zone on F.Cu, net Net-(D6-A)
Other:
- board text removed: "{ "ViaStitching": "0.2", "stitch_zone_0": { "HSpacing": "1.5", "VSpacing": "1.5", "HOffset": "1", "VOffset": "1", "Clearance": "0.5", "Randomize": false } }"

Commit message: pcbs final update
Parts:
- added D17: LED, LED_THT:LED_D3.0mm, F.Cu at (135.5, 82.0)
- added R32: 100, Resistor_SMD:R_0603_1608Metric, F.Cu at (134.5, 77.5)
Routing:
- net /Microcontroller/GPIO39: track 0.00 -> 19.3 mm, vias 0 -> 4
- net Net-(D17-A): track 0.00 -> 2.03 mm
- net /Microcontroller/GPIO16: track 42.0 -> 41.3 mm
- net GND: vias 366 -> 243

Commit message: pcbs update
Parts:
- moved C1 44.0 mm to (157.9, 87.4)
- moved C2 44.0 mm to (157.9, 85.9)
- moved C3 44.0 mm to (154.2, 86.7)
- moved R1 44.0 mm to (155.7, 86.7)
- moved J5 44.0 mm to (144.9, 105.1)
- moved K3 44.0 mm to (113.6, 113.2)
- moved K4 44.0 mm to (113.6, 125.4)
- moved R16 44.0 mm to (145.2, 110.3)
- moved R18 44.0 mm to (148.7, 105.6)
- moved R4 44.0 mm to (142.4, 87.9)
- moved R7 44.0 mm to (142.4, 90.9)
- moved C11 44.0 mm to (170.5, 84.8)
- moved C14 44.0 mm to (164.5, 84.8)
- moved C5 44.0 mm to (180.6, 120.3)
- moved C6 44.0 mm to (180.5, 118.8)
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